File: Training/Renganathan_Laasya/timer.sch (EAGLE design)
At the start: 8 parts, among them IC1 NE555, J1 1X2-3.5MM

Commit message: updated training project
thanks
Parts:
- 9V: value 1X2-3.5MM -> VCC+
- R3: value 1k -> (none)
- renumbered J1 to 9V
Connections:
- net VCC+ renamed VCC9V
Changed lines of the file:
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@@
 <part name="C2" library="SparkFun-Passives" deviceset="CAP" device="PTH" value="10n"/>
 <part name="LED1" library="adafruit" deviceset="LED" device="5MM" value="RED"/>
-<part name="J1" library="adafruit" deviceset="1X2" device="-3.5MM"/>
-<part name="R3" library="SparkFun-Resistors" deviceset="RESISTOR" device="AXIAL-0.3" value="1k"/>
+<part name="9V" library="adafruit" deviceset="1X2" device="-3.5MM" value="VCC+"/>
+<part name="R3" library="SparkFun-Resistors" deviceset="RESISTOR" device="AXIAL-0.3" value="
+                                                                                            "/>
+<part name="GND1" library="SparkFun-Aesthetics" deviceset="GND" device=""/>
+<part name="SUPPLY1" library="SparkFun-Aesthetics" deviceset="VCC" device="" value="9V"/>
 </parts>
 <sheets>
@@
 <instance part="C2" gate="G$1" x="76.2" y="25.4"/>
 <instance part="LED1" gate="G$1" x="88.9" y="33.02"/>
-<instance part="J1" gate="G$1" x="25.4" y="66.04" rot="MR90"/>
+<instance part="9V" gate="G$1" x="25.4" y="66.04" rot="MR90"/>
 <instance part="R3" gate="G$1" x="88.9" y="48.26" rot="R270"/>
+<instance part="GND1" gate="1" x="25.4" y="15.24"/>
+<instance part="SUPPLY1" gate="G$1" x="33.02" y="60.96"/>
 </instances>
 <busses>
@@
 </segment>
 </net>
-<net name="VCC+" class="0">
-<segment>
-<pinref part="R1" gate="G$1" pin="1"/>
-<wire x1="35.56" y1="58.42" x2="35.56" y2="60.96" width="0.1524" layer="91"/>
-<pinref part="J1" gate="G$1" pin="1"/>
-<wire x1="35.56" y1="60.96" x2="27.94" y2="60.96" width="0.1524" layer="91"/>
-<pinref part="IC1" gate="G$1" pin="VCC+"/>
-<wire x1="71.12" y1="45.72" x2="71.12" y2="60.96" width="0.1524" layer="91"/>
-<wire x1="71.12" y1="60.96" x2="35.56" y2="60.96" width="0.1524" layer="91"/>
-<junction x="35.56" y="60.96"/>
-<pinref part="IC1" gate="G$1" pin="/RES"/>
-<wire x1="71.12" y1="43.18" x2="76.2" y2="43.18" width="0.1524" layer="91"/>
-<wire x1="76.2" y1="43.18" x2="76.2" y2="60.96" width="0.1524" layer="91"/>
-<wire x1="76.2" y1="60.96" x2="71.12" y2="60.96" width="0.1524" layer="91"/>
-<junction x="71.12" y="60.96"/>
-</segment>
-</net>
 <net name="N$7" class="0">
 <segment>
@@
 <pinref part="LED1" gate="G$1" pin="C"/>
 <wire x1="88.9" y1="27.94" x2="88.9" y2="17.78" width="0.1524" layer="91"/>
-<pinref part="J1" gate="G$1" pin="2"/>
+<pinref part="9V" gate="G$1" pin="2"/>
 <wire x1="88.9" y1="17.78" x2="76.2" y2="17.78" width="0.1524" layer="91"/>
 <wire x1="76.2" y1="17.78" x2="71.12" y2="17.78" width="0.1524" layer="91"/>
@@
 <wire x1="35.56" y1="20.32" x2="35.56" y2="17.78" width="0.1524" layer="91"/>
 <junction x="35.56" y="17.78"/>
+<pinref part="GND1" gate="1" pin="GND"/>
+<junction x="25.4" y="17.78"/>
 </segment>
 </net>
@@
 </segment>
 </net>
+<net name="VCC9V" class="0">
+<segment>
+<pinref part="R1" gate="G$1" pin="1"/>
+<wire x1="35.56" y1="58.42" x2="35.56" y2="60.96" width="0.1524" layer="91"/>
+<pinref part="9V" gate="G$1" pin="1"/>
+<wire x1="35.56" y1="60.96" x2="33.02" y2="60.96" width="0.1524" layer="91"/>
+<pinref part="IC1" gate="G$1" pin="VCC+"/>
+<wire x1="33.02" y1="60.96" x2="27.94" y2="60.96" width="0.1524" layer="91"/>
+<wire x1="71.12" y1="45.72" x2="71.12" y2="60.96" width="0.1524" layer="91"/>
+<wire x1="71.12" y1="60.96" x2="35.56" y2="60.96" width="0.1524" layer="91"/>
+<junction x="35.56" y="60.96"/>
+<pinref part="IC1" gate="G$1" pin="/RES"/>
+<wire x1="71.12" y1="43.18" x2="76.2" y2="43.18" width="0.1524" layer="91"/>
+<wire x1="76.2" y1="43.18" x2="76.2" y2="60.96" width="0.1524" layer="91"/>
+<wire x1="76.2" y1="60.96" x2="71.12" y2="60.96" width="0.1524" layer="91"/>
+<junction x="71.12" y="60.96"/>
+<pinref part="SUPPLY1" gate="G$1" pin="VCC"/>
+<junction x="33.02" y="60.96"/>
+</segment>
+</net>

Commit message: Update timer.sch
Parts:
- R3: value (none) -> 510
Changed lines of the file:
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@@
 <part name="LED1" library="adafruit" deviceset="LED" device="5MM" value="RED"/>
 <part name="9V" library="adafruit" deviceset="1X2" device="-3.5MM" value="VCC+"/>
-<part name="R3" library="SparkFun-Resistors" deviceset="RESISTOR" device="AXIAL-0.3" value="
-                                                                                            "/>
+<part name="R3" library="SparkFun-Resistors" deviceset="RESISTOR" device="AXIAL-0.3" value="510"/>
 <part name="GND1" library="SparkFun-Aesthetics" deviceset="GND" device=""/>
 <part name="SUPPLY1" library="SparkFun-Aesthetics" deviceset="VCC" device="" value="9V"/>
