File: Full_TDS/full_tds.sch (EAGLE design)
At the start: 68 parts, among them IC1 MCP1702, Q1 NFET, Q2 PFET, Q3 NFET, Q4 PFET, Q9 8MHz, U1 MPL3115A2LGA8, U2 ADXL345PATRICK, U3 ATMEGA328P_PDIP, U4 FT232RLSSOP, X2 USBSMD

Commit message: full sch
Connections:
- removed net GND: C1.2, C2.-, C3.2, C4.-, C5.2, C6.2, CIO.2, U1.GND, U2.GND@2, U2.GND@4, U2.GND@5, U2.SDO
- removed net VCC_3.3V: C1.1, C2.+, C3.1, C4.+, C6.1, CIO.1, R1.2, R2.2, U1.VDD, U1.VDDIO, U2.CS, U2.VDD, U2.VSS
- net 3.3V: now also C1.1, C2.+, C3.1, C4.+, C6.1, CIO.1, R1.2, R2.2, U1.VDD, U1.VDDIO, U2.CS, U2.VDD, U2.VSS
- net GND-ISO: now also C1.2, C2.-, C3.2, C4.-, C5.2, C6.2, CIO.2, U1.GND, U2.GND@2, U2.GND@4, U2.GND@5, U2.SDO
Other:
- note removed: "Power Distribution Module"
- note removed: "State Control Module"
- moved on the sheet: C1, C10, C2, C3, C4, C5, C6, C7, C8, C9, CIO, D1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
