File: Full_TDS/full_tds.sch (EAGLE design)
At the start: 68 parts, among them IC1 MCP1702, Q5 8MHz, SW1 MAIN, SW2 PI, SW3 SENSOR, U2 FT232RLSSOP, U3 ADXL345PATRICK, U4 MPL3115A2LGA8, U5 ATMEGA328P_TQFP

Commit message: Schematic should be ready, starting board
Parts:
- removed JP3: POWER, SparkFun-Connectors:M02PTH
- removed POWER, SCM: (no value), SparkFun-Connectors:M02PTH
- added U$3: RASPBERRY-PI-HEADER2B, custom:RASPBERRY-PI-HEADER2B
Connections:
- new net A0: U$3.GP5, U5.PC0(ADC0)
- net 3.3V: no longer JP3.1
- net GND-ISO: now also U$3.GND@14, U$3.GND@20, U$3.GND@25, U$3.GND@30, U$3.GND@34, U$3.GND@39, U$3.GND@6, U$3.GND@9; no longer JP3.2, POWER.2
- net MISO: now also U$3.MISO
- net MOSI: now also U$3.MOSI
- net PI_5V: now also U$3.5V@2
- net SCL: no longer SCM.1
- net SCLK: now also U$3.SCLK
- net SDA: no longer SCM.2
- net SENSOR_POWER: no longer POWER.1
- net SS: now also U$3.CE0
Other:
- moved on the sheet: C1, C12, C13, C14, C15, C16, C17, C18, C19, C2, C20, C5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

Commit message: Some schematic adjustments and board progress
Parts:
- removed JP1: GPIO, SparkFun-Connectors:M03PTH
- removed JP4: ACCEL, SparkFun-Connectors:M02PTH
- removed JP5: ALT, SparkFun-Connectors:M02PTH
- removed JP8: USB-MICROB, SparkFun-Connectors:USB-MICROB
- removed SENSOR, STATE_CONTROLLER: (no value), SparkFun-Connectors:M02PTH
- added 3.3V: (no value), SparkFun-Connectors:M02PTH
- F1, F2: device fuse:FUSEPICOFUSE -> SparkFun-Fuses:PPTC_HALF-AMP
- F3: device fuse:PICOFUSE -> SparkFun-Fuses:PPTC_HALF-AMP
Connections:
- removed net USB_D+: JP8.D+, U2.USBDP
- removed net USB_D-: JP8.D-, U2.USBDM
- removed net VBUS: C2.1, C5.1, C6.2, JP8.VBUS, U2.VCC
- new net D+: JP7.D+, U2.USBDP
- new net D-: JP7.D-, U2.USBDM
- net 3.3V: now also 3.3V.1; no longer STATE_CONTROLLER.1
- net 5V_RAW: now also C2.1, C5.1, C6.2, U2.VCC
- net ACCEL_INT1: no longer JP4.1
- net ACCEL_INT2: no longer JP4.2
- net ALT_INT1: no longer JP5.1
- net ALT_INT2: no longer JP5.2
- net GND-ISO: now also 3.3V.2; no longer JP8.GND, SENSOR.2, STATE_CONTROLLER.2
- net INT0: no longer JP1.1
- net INT1: no longer JP1.2
- net IO4: no longer JP1.3
- net SENSOR_POWER: no longer SENSOR.1
Other:
- moved on the sheet: C6, CNTRL_INPUTS, JP2, JP9, PI

Commit message: Board possibly done, need more checking
Parts:
- added R2: 0, SparkFun-Resistors:RESISTOR1206
Connections:
- new net FT232_VCC: C2.1, C5.1, C6.2, R2.1, U$2.S1(P), U2.VCC
- net 5V: now also R2.2; no longer U$2.S1(P)
- net 5V_RAW: no longer C2.1, C5.1, C6.2, U2.VCC
- net PI_5V: now also U$3.5V@4
