File: Full_TDS/full_tds.sch (EAGLE design)
At the start: 62 parts, among them IC1 MCP1702, Q5 8MHz, SW1 MAIN, SW2 PI, SW3 SENSOR, U2 FT232RLSSOP, U3 ADXL345PATRICK, U4 MPL3115A2LGA8, U5 ATMEGA328P_TQFP

Commit message: Full TDS rev2
Parts:
- removed D3: TVS, SparkFun-DiscreteSemi:DIODEPTH
- added R3, R4: 470, SparkFun-Passives:RESISTOR1206
- added STATUS1: Green, adafruit:LEDCHIPLED_1206
- added STATUS2: Blue, adafruit:LEDCHIPLED_1206
Connections:
- net N$13 renamed FUSE_DIODE_PI
- net N$18 renamed XTAL1
- net N$19 renamed XTAL2
- net N$21 renamed PD5
- net N$23 renamed PD6
- net N$24 renamed PD7
- net N$3 renamed PI_P_DRAIN
- net N$4 renamed VCCIO
- net N$5 renamed SENS_N_DRAIN
- net N$6 renamed SENS_P_DRAIN
- net N$7 renamed PI_N_DRAIN
- removed net INT0: U5.PD2(INT0)
- removed net INT1: U5.PD3(INT1)
- removed net IO4: U5.PD4(XCK/T0)
- removed net N$22: C19.2, C20.2, U5.AGND, U5.GND@3, U5.GND@5
- new net A1: U$3.GP6, U5.PC1(ADC1)
- new net A2: U$3.GP12, U5.PC2(ADC2)
- new net GP13: R3.1, U$3.GP13
- new net GP16: R4.1, U$3.GP16
- new net N$10: R4.2, STATUS2.A
- new net N$11: R3.2, STATUS1.A
- new net PI_3.3V: U$3.3.3V@1, U$3.3.3V@17
- net 5V: no longer D3.C
- net GND-ISO: now also C19.2, C20.2, STATUS1.C, STATUS2.C, U5.AGND, U5.GND@3, U5.GND@5; no longer D3.A
Other:
- moved on the sheet: R16, R17

Commit message: New TDS rev
Parts:
- added SW4: RESET, special:SW_DIP-1
Connections:
- net GND-ISO: now also SW4.2
- net RESET: now also SW4.1
Changed lines of the file:
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@@
 <part name="STATUS2" library="adafruit" deviceset="LED" device="CHIPLED_1206" value="Blue"/>
 <part name="GND-ISO18" library="SparkFun-Aesthetics" deviceset="GND-ISO" device=""/>
+<part name="SW4" library="special" deviceset="SW_DIP-1" device="" value="RESET"/>
+<part name="GND-ISO21" library="SparkFun-Aesthetics" deviceset="GND-ISO" device=""/>
 </parts>
 <sheets>
@@
 <attribute name="VALUE" x="-22.86" y="205.74" size="1.778" layer="96"/>
 </instance>
+<instance part="SW4" gate="G$1" x="-60.96" y="106.68" rot="R90"/>
+<instance part="GND-ISO21" gate="G$1" x="-60.96" y="93.98"/>
 </instances>
 <busses>
@@
 <junction x="-17.78" y="215.9"/>
 </segment>
+<segment>
+<pinref part="GND-ISO21" gate="G$1" pin="GND-ISO"/>
+<pinref part="SW4" gate="G$1" pin="2"/>
+<wire x1="-60.96" y1="96.52" x2="-60.96" y2="99.06" width="0.1524" layer="91"/>
+</segment>
 </net>
 <net name="SS" class="0">
@@
 <pinref part="R15" gate="G$1" pin="1"/>
 <wire x1="-43.18" y1="86.36" x2="-43.18" y2="93.98" width="0.1524" layer="91"/>
-<wire x1="-43.18" y1="86.36" x2="-50.8" y2="86.36" width="0.1524" layer="91"/>
+<wire x1="-43.18" y1="86.36" x2="-53.34" y2="86.36" width="0.1524" layer="91"/>
 <junction x="-43.18" y="86.36"/>
-<wire x1="-50.8" y1="86.36" x2="-50.8" y2="88.9" width="0.1524" layer="91"/>
-<label x="-50.8" y="88.9" size="1.27" layer="95" rot="R90" xref="yes"/>
+<label x="-53.34" y="86.36" size="1.27" layer="95" rot="R180" xref="yes"/>
 <pinref part="U5" gate="U$1" pin="VCC@6"/>
 <wire x1="-17.78" y1="86.36" x2="-17.78" y2="83.82" width="0.1524" layer="91"/>
@@
 <pinref part="C18" gate="G$1" pin="2"/>
 <pinref part="U5" gate="U$1" pin="PC6(/RESET)"/>
-<wire x1="-27.94" y1="93.98" x2="-20.32" y2="93.98" width="0.1524" layer="91"/>
+<wire x1="-27.94" y1="93.98" x2="-22.86" y2="93.98" width="0.1524" layer="91"/>
 <pinref part="R15" gate="G$1" pin="2"/>
+<wire x1="-22.86" y1="93.98" x2="-20.32" y2="93.98" width="0.1524" layer="91"/>
 <wire x1="-20.32" y1="93.98" x2="-17.78" y2="93.98" width="0.1524" layer="91"/>
 <wire x1="-27.94" y1="93.98" x2="-33.02" y2="93.98" width="0.1524" layer="91"/>
@@
 <junction x="-20.32" y="93.98"/>
 <label x="-20.32" y="101.6" size="1.27" layer="95" rot="R90" xref="yes"/>
-</segment>
-</net>
+<pinref part="SW4" gate="G$1" pin="1"/>
+<wire x1="-60.96" y1="114.3" x2="-22.86" y2="114.3" width="0.1524" layer="91"/>
+<wire x1="-22.86" y1="114.3" x2="-22.86" y2="93.98" width="0.1524" layer="91"/>
+<junction x="-22.86" y="93.98"/>
+</segment>
+</net>

Commit message: hi
Connections:
- net DTR: no longer U2.DTR
Other:
- moved on the sheet: 3.3V, C1, C10, C11, C12, C13, C14, C15, C16, C17, C2, C5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
