File: Full_TDS/full_tds.brd (EAGLE design)
At the start: 68.2 x 41.9 mm, 69 parts, among them IC1 MCP1702, Q1 NFET, Q2 PFET, Q3 NFET, Q4 PFET, Q5 8MHz, U2 FT232RLSSOP, U3 ADXL345PATRICK, U4 MPL3115A2LGA8, U5 ATMEGA328P_TQFP, X2 USBSMD

Commit message: Schem touch up
Connections:
- net PI_PWR_CNTRL: now also U5.13
- net SENSOR_PWR_CNTRL: now also U5.12
Changed lines of the file:
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@@
 <contactref element="Q1" pad="1"/>
 <contactref element="CNTRL_INPUTS" pad="2"/>
-<wire x1="41.91" y1="-38.1" x2="46.99" y2="0" width="0" layer="19" extent="1-1"/>
-<wire x1="42.062" y1="-66.04" x2="41.91" y2="-38.1" width="0" layer="19" extent="1-1"/>
+<contactref element="U5" pad="13"/>
+<wire x1="42.062" y1="-66.04" x2="-12.3" y2="-149.0726" width="0" layer="19" extent="1-1"/>
+<wire x1="41.91" y1="-38.1" x2="42.062" y2="-66.04" width="0" layer="19" extent="1-1"/>
+<wire x1="46.99" y1="0" x2="41.91" y2="-38.1" width="0" layer="19" extent="1-1"/>
 </signal>
 <signal name="N$12">
@@
 <contactref element="Q3" pad="1"/>
 <contactref element="CNTRL_INPUTS" pad="1"/>
+<contactref element="U5" pad="12"/>
+<wire x1="2.54" y1="-54.61" x2="-13.1" y2="-149.0726" width="0" layer="19" extent="1-1"/>
 <wire x1="47.142" y1="-66.04" x2="2.54" y2="-54.61" width="0" layer="19" extent="1-1"/>
 <wire x1="44.45" y1="0" x2="47.142" y2="-66.04" width="0" layer="19" extent="1-1"/>

Commit message: Replaced capacitors with 1206
Parts:
- C1, C18, C2: value 0.1uF -> .1 uF; device SparkFun-Capacitors:CAP-PTH-SMALL -> SparkFun-Capacitors:1206
- C10, C11, C19, C20, C6: device SparkFun-Capacitors:CAP-PTH-SMALL -> SparkFun-Capacitors:1206
- C12, C14, CIO: value 0.1uF -> .1 uF; device SparkFun-Passives:CAP-PTH-SMALL -> SparkFun-Capacitors:1206
- C13, C15, C5, C9: device SparkFun-Passives:CPOL-RADIAL-10UF-25V -> adafruit:C1206
- C16: value 0.1uF -> .1 uF
- C8: device SparkFun-Passives:CAP-PTH-SMALL -> SparkFun-Capacitors:1206
Routing:
- net GND-ISO: track 90.8 -> 93.8 mm
- net N$4: track 26.1 -> 27.3 mm
- net VBUS: track 72.4 -> 73.5 mm

Commit message: Replaced transistors with SMD part
Parts:
- removed Q1, Q3: NFET, User-Submitted:TO220V
- removed Q2, Q4: PFET, User-Submitted:TO220V
- removed X2: USBSMD, SparkFun-Connectors:USB-MINIB
- added JP8: USB-MICROB, SparkFun-Connectors:USB-MICROB
- added JP9: I2C, SparkFun-Connectors:1X02
- added U$1, U$2: DMC3021LSD-13, custom:SOIC-8
- C1, C10, C11, C12, C14, C18, C2, C8, CIO: value .1 uF -> 0.1 uF
- C16: value .1 uF -> 0.1 uF; device SparkFun-Passives:CAP-PTH-SMALL -> SparkFun-Capacitors:1206
- C17: value 1uF -> 1.0uF; device SparkFun-Passives:CAP-PTH-SMALL -> SparkFun-Capacitors:1206
- LED1, LED2, LED6, LED7, LED8: device adafruit:LED5MM -> adafruit:CHIPLED_1206
- SW1: value (none) -> MAIN
- SW2: value (none) -> PI
- SW3: value (none) -> SENSOR
Connections:
- removed net INT2: U4.5
- removed net N$12: F1.1, Q2.2, R9.2, SW2.1
- removed net N$14: Q3.2, Q4.1, R14.1
- removed net N$15: F2.1, Q4.2, R13.2, SW3.1
- new net ACCEL_INT1: JP4.1, U3.8
- new net ACCEL_INT2: JP4.2, U3.9
- new net ALT_INT1: JP5.1, U4.6
- new net ALT_INT2: JP5.2, U4.5
- new net N$5: R14.1, U$1.4, U$1.7, U$1.8
- new net N$6: F2.1, R13.2, SW3.1, U$1.5, U$1.6
- new net N$7: R10.1, U$2.4, U$2.7, U$2.8
- net 3.3V: now also U$1.3; no longer Q4.3
- net 5V: now also U$2.3; no longer Q2.3
- net GND-ISO: now also JP8.GND, JP8.MT1, JP8.MT2, LED6.C, LED7.C, LED8.C, U$1.1, U$2.1; no longer LED6.K, LED7.K, LED8.K, Q1.3, Q3.3, X2.GND
- net INT1: no longer U4.6
- net N$3: now also F1.1, R9.2, SW2.1, U$2.5, U$2.6; no longer Q1.2, Q2.1, R10.1
- net PI_PWR_CNTRL: now also U$2.2; no longer Q1.1
- net RXLED: now also LED2.C; no longer LED2.K
- net SCL: now also JP9.2; no longer JP4.2, JP5.2
- net SDA: now also JP9.1; no longer JP4.1, JP5.1
- net SENSOR_PWR_CNTRL: now also U$1.2; no longer Q3.1
- net TXLED: now also LED1.C; no longer LED1.K
- net USB_D+: now also JP8.D+; no longer X2.D+
- net USB_D-: now also JP8.D-; no longer X2.D-
- net VBUS: now also JP8.VBUS; no longer X2.VBUS
Routing:
- net GND-ISO: track 93.8 -> 0.00 mm, vias 1 -> 0
- net VBUS: track 73.5 -> 0.00 mm, vias 1 -> 0
- net USB_D+: track 59.6 -> 0.00 mm
- net MOSI: track 46.1 -> 0.00 mm
- net SS: track 41.5 -> 0.00 mm
- net SCLK: track 38.6 -> 0.00 mm
- net SCL: track 37.9 -> 0.00 mm
- net 3.3V: track 37.0 -> 0.00 mm, vias 1 -> 0
- net MISO: track 34.5 -> 0.00 mm
- net TXO: track 34.0 -> 0.00 mm, vias 1 -> 0
- net RXI: track 32.6 -> 0.00 mm, vias 1 -> 0
- net USB_D-: track 30.7 -> 0.00 mm
- net N$4: track 27.3 -> 0.00 mm, vias 1 -> 0
- net N$2: track 25.5 -> 0.00 mm
- net TXLED: track 21.1 -> 0.00 mm
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
Commit message: Schematic should be ready, starting board
Parts:
- removed JP3: POWER, SparkFun-Connectors:1X02
- removed POWER, SCM: (no value), SparkFun-Connectors:1X02
- added U$3: RASPBERRY-PI-HEADER2B, custom:2X20-NOSILK
- moved U$1 342.9 mm to (33.0, 41.9)
- moved U$2 321.9 mm to (29.2, 19.1)
- moved JP9 317.4 mm to (52.1, 16.5)
- moved JP8 315.7 mm to (57.1, 25.4)
- moved LED8 314.1 mm to (53.3, 40.6)
- moved LED7 277.5 mm to (26.7, 27.9)
- moved LED6 275.9 mm to (61.0, 33.0)
- moved R16 267.4 mm to (33.0, 49.5)
- moved R17 267.1 mm to (26.7, 49.5)
- moved R18 266.8 mm to (20.3, 49.5)
- moved R19 266.5 mm to (14.0, 49.5)
- moved R20 266.3 mm to (7.62, 49.5)
- moved C19 254.2 mm to (63.5, 52.1), turned to 90 degrees
- moved C20 236.4 mm to (33.0, 25.4)
- moved Q5 220.4 mm to (11.4, 43.2)
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Connections:
- new net A0: U$3.29, U5.23
- net 3.3V: now also U$3.1, U$3.17; no longer JP3.1
- net 5V: now also U$3.4
- net GND-ISO: now also U$3.14, U$3.20, U$3.25, U$3.30, U$3.34, U$3.39, U$3.6, U$3.9; no longer JP3.2, POWER.2
- net MISO: now also U$3.21
- net MOSI: now also U$3.19
- net PI_5V: now also U$3.2
- net SCL: no longer SCM.1
- net SCLK: now also U$3.23
- net SDA: no longer SCM.2
- net SENSOR_POWER: no longer POWER.1
- net SS: now also U$3.24
Other:
- board size 68.2 x 41.9 mm -> 69.5 x 52.1 mm
- board text removed: "F. Kummer SCM v1"

Commit message: Some schematic adjustments and board progress
Parts:
- removed JP1: GPIO, SparkFun-Connectors:1X03
- removed JP4: ACCEL, SparkFun-Connectors:1X02
- removed JP5: ALT, SparkFun-Connectors:1X02
- removed JP8: USB-MICROB, SparkFun-Connectors:USB-MICROB
- removed SENSOR, STATE_CONTROLLER: (no value), SparkFun-Connectors:1X02
- added 3.3V: (no value), SparkFun-Connectors:1X02
- F1, F2, F3: device fuse:PICOFUSE -> SparkFun-Fuses:1206
- moved SW2 70.8 mm to (78.7, 8.89)
- moved F3 70.1 mm to (74.9, 20.3)
- moved C17 68.4 mm to (78.7, 35.6), turned to 90 degrees
- moved R15 65.1 mm to (78.7, 40.6)
- moved F1 57.7 mm to (78.7, 19.1)
- moved C5 50.4 mm to (21.6, 5.08)
- moved SW3 50.3 mm to (64.8, 17.8)
- moved D1 44.3 mm to (53.3, 16.5), turned to 270 degrees
- moved C6 43.1 mm to (17.8, 10.2)
- moved C2 42.7 mm to (21.6, 10.2)
- moved C1 38.1 mm to (17.8, 5.08), turned to 90 degrees
- moved R1 36.9 mm to (27.9, 21.6), turned to 90 degrees
- moved LED1 35.4 mm to (24.1, 27.9)
- moved R5 31.2 mm to (31.8, 21.6), turned to 90 degrees
- moved LED7 30.7 mm to (54.6, 40.6)
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Connections:
- removed net USB_D+: JP8.D+, U2.15
- removed net USB_D-: JP8.D-, U2.16
- removed net VBUS: C2.1, C5.1, C6.2, JP8.VBUS, U2.20
- new net D+: JP7.D+, U2.15
- new net D-: JP7.D-, U2.16
- net 3.3V: now also 3.3V.1; no longer STATE_CONTROLLER.1
- net 5V_RAW: now also C2.1, C5.1, C6.2, U2.20
- net ACCEL_INT1: no longer JP4.1
- net ACCEL_INT2: no longer JP4.2
- net ALT_INT1: no longer JP5.1
- net ALT_INT2: no longer JP5.2
- net GND-ISO: now also 3.3V.2; no longer JP8.GND, JP8.MT1, JP8.MT2, SENSOR.2, STATE_CONTROLLER.2
- net INT0: no longer JP1.1
- net INT1: no longer JP1.2
- net IO4: no longer JP1.3
- net SENSOR_POWER: no longer SENSOR.1

Commit message: Board possibly done, need more checking
Parts:
- added R2: 0, SparkFun-Resistors:1206
- moved C19 61.8 mm to (21.6, 40.6)
- moved C18 48.4 mm to (31.8, 49.5), turned to 180 degrees
- moved U$3 48.3 mm to (73.7, 7.62), turned to 180 degrees
- moved JP9 45.6 mm to (61.0, 55.9), turned to 180 degrees
- moved C20 43.7 mm to (25.4, 49.5)
- moved LED6 39.9 mm to (48.3, 44.5), turned to 90 degrees
- moved R15 35.4 mm to (44.5, 49.5)
- moved IC1 29.6 mm to (52.1, 31.8)
- moved F1 25.2 mm to (59.7, 35.6)
- moved C16 25.0 mm to (54.6, 41.9), turned to 270 degrees
- moved F2 24.4 mm to (66.0, 35.6)
- moved LED8 24.3 mm to (48.3, 36.8), turned to 90 degrees
- moved R20 23.4 mm to (44.5, 33.0)
- moved C11 22.2 mm to (77.5, 48.3), turned to 90 degrees
- moved SW2 21.8 mm to (66.0, 26.7)
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Connections:
- new net FT232_VCC: C2.1, C5.1, C6.2, R2.1, U$2.3, U2.20
- net 5V: now also R2.2; no longer U$2.3, U$3.4
- net 5V_RAW: no longer C2.1, C5.1, C6.2, U2.20
- net PI_5V: now also U$3.4
Routing:
- net GND-ISO: track 0.00 -> 419.8 mm, vias 0 -> 6
- net 3.3V: track 0.00 -> 211.1 mm, vias 0 -> 5
- net 5V: track 0.00 -> 138.8 mm, vias 0 -> 1
- net MOSI: track 0.00 -> 113.3 mm, vias 0 -> 3
- net MISO: track 0.00 -> 102.6 mm, vias 0 -> 3
- net SCLK: track 0.00 -> 91.2 mm, vias 0 -> 5
- net PI_5V: track 0.00 -> 78.6 mm, vias 0 -> 1
- net SDA: track 0.00 -> 77.0 mm
- net SENSOR_PWR_CNTRL: track 0.00 -> 66.0 mm, vias 0 -> 3
- net 5V_RAW: track 0.00 -> 64.9 mm, vias 0 -> 1
- net SS: track 0.00 -> 61.0 mm, vias 0 -> 2
- net PI_PWR_CNTRL: track 0.00 -> 56.9 mm, vias 0 -> 3
- net N$6: track 0.00 -> 56.5 mm, vias 0 -> 3
- net SCL: track 0.00 -> 54.0 mm, vias 0 -> 4
- net N$3: track 0.00 -> 53.3 mm, vias 0 -> 2
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Other:
- board size 69.5 x 52.1 mm -> 64.4 x 55.9 mm
