File: Full_TDS/full_tds.brd (EAGLE design)
At the start: 64.4 x 55.9 mm, 62 parts, among them IC1 MCP1702, Q5 8MHz, SW1 MAIN, SW2 PI, SW3 SENSOR, U2 FT232RLSSOP, U3 ADXL345PATRICK, U4 MPL3115A2LGA8, U5 ATMEGA328P_TQFP

Commit message: Full TDS rev2
Parts:
- removed D3: TVS, SparkFun-DiscreteSemi:DIODE-1N4001
- added R3, R4: 470, SparkFun-Passives:1206
- added STATUS1: Green, adafruit:CHIPLED_1206
- added STATUS2: Blue, adafruit:CHIPLED_1206
- moved D1 6.35 mm to (64.8, 17.8)
Connections:
- net N$13 renamed FUSE_DIODE_PI
- net N$18 renamed XTAL1
- net N$19 renamed XTAL2
- net N$21 renamed PD5
- net N$23 renamed PD6
- net N$24 renamed PD7
- net N$3 renamed PI_P_DRAIN
- net N$4 renamed VCCIO
- net N$5 renamed SENS_N_DRAIN
- net N$6 renamed SENS_P_DRAIN
- net N$7 renamed PI_N_DRAIN
- removed net INT0: U5.32
- removed net INT1: U5.1
- removed net IO4: U5.2
- removed net N$22: C19.2, C20.2, U5.21, U5.3, U5.5
- new net A1: U$3.31, U5.24
- new net A2: U$3.32, U5.25
- new net GP13: R3.1, U$3.33
- new net GP16: R4.1, U$3.36
- new net N$10: R4.2, STATUS2.A
- new net N$11: R3.2, STATUS1.A
- new net PI_3.3V: U$3.1, U$3.17
- net 3.3V: no longer U$3.1, U$3.17
- net 5V: no longer D3.C
- net GND-ISO: now also C19.2, C20.2, STATUS1.C, STATUS2.C, U5.21, U5.3, U5.5; no longer D3.A
Routing:
- net A1: track 0.00 -> 76.6 mm, vias 0 -> 1
- net A2: track 0.00 -> 60.6 mm, vias 0 -> 1
- net GP13: track 0.00 -> 36.8 mm
- net GND-ISO: track 419.8 -> 453.4 mm
- net N$22: track 33.4 -> 0.00 mm
- net GP16: track 0.00 -> 31.2 mm
- net 5V: track 138.8 -> 109.6 mm, vias 1 -> 5
- net MOSI: track 113.3 -> 84.9 mm, vias 3 -> 6
- net SCLK: track 91.2 -> 119.2 mm, vias 5 -> 1
- net A0: track 38.9 -> 66.8 mm, vias 2 -> 1
- net PI_3.3V: track 0.00 -> 21.3 mm
- net 3.3V: track 211.1 -> 191.0 mm, vias 5 -> 2
- net PI_5V: track 78.6 -> 97.7 mm
- net MISO: track 102.6 -> 121.1 mm, vias 3 -> 4
- net 5V_RAW: track 64.9 -> 47.0 mm, vias 1 -> 4
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Other:
- board text added: "SCL"
- board text added: "SDA"

Commit message: New TDS rev
Parts:
- added SW4: RESET, special:EDG-01
- moved C18 8.91 mm to (22.9, 48.9)
- moved R4 6.35 mm to (66.0, 10.8)
- moved STATUS2 6.35 mm to (66.0, 14.0)
- moved R15 6.02 mm to (50.2, 51.4)
- moved R16 6.02 mm to (43.8, 51.4)
- moved C20 4.07 mm to (22.9, 52.7)
- moved R3 3.81 mm to (73.7, 10.8)
- moved STATUS1 3.81 mm to (73.7, 14.0)
- moved U$1 1.27 mm to (48.3, 14.0)
- moved U$2 1.27 mm to (35.6, 14.0)
- flipped SW1 to the top
Connections:
- net GND-ISO: now also SW4.2
- net RESET: now also SW4.1
Routing:
- net MOSI: track 84.9 -> 124.4 mm, vias 6 -> 2
- net A1: track 76.6 -> 41.7 mm
- net RESET: track 26.0 -> 53.5 mm, vias 0 -> 2
- net PI_5V: track 97.7 -> 77.2 mm, vias 1 -> 2
- net A0: track 66.8 -> 46.6 mm, vias 1 -> 3
- net TXO: track 44.2 -> 30.5 mm, vias 0 -> 2
- net SDA: track 75.4 -> 63.2 mm, vias 0 -> 4
- net PI_PWR_CNTRL: track 71.3 -> 60.5 mm, vias 2 -> 5
- net MISO: track 121.1 -> 111.3 mm, vias 4 -> 3
- net SCL: track 62.9 -> 53.5 mm, vias 4 -> 6
- net SCLK: track 119.2 -> 109.8 mm, vias 1 -> 4
- net GND-ISO: track 453.4 -> 444.4 mm, vias 6 -> 5
- net GP13: track 36.8 -> 45.7 mm, vias 0 -> 1
- net A2: track 60.6 -> 69.2 mm, vias 1 -> 3
- net SS: track 58.3 -> 66.5 mm, vias 1 -> 3
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Other:
- board text added: "CRT"
- board text added: "TDS rev2"

Commit message: hi
Connections:
- net DTR: no longer U2.2
Changed lines of the file:
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@@
 </signal>
 <signal name="DTR">
-<contactref element="U2" pad="2"/>
 <contactref element="C18" pad="1"/>
 <wire x1="16.0782" y1="23.9268" x2="16.6116" y2="23.9268" width="0.1524" layer="1"/>
@@
 <wire x1="23.1648" y1="49.9872" x2="23.1648" y2="53.0352" width="0.1524" layer="1"/>
 <wire x1="24.2316" y1="48.9204" x2="23.1648" y2="49.9872" width="0.1524" layer="1"/>
-<wire x1="16.6116" y1="23.9268" x2="16.664" y2="23.895" width="0.1524" layer="1"/>
 <wire x1="24.2316" y1="48.9204" x2="24.26" y2="48.895" width="0.1524" layer="1"/>
 </signal>
