File: RCS/RCSfullschematic.sch (EAGLE design)
At the start: 72 parts, among them IC1 ILD213T, IC2 FT232RL, J2 MOTOR, J4 POWER, J5 SENSORS, J7 USB-MICROB, Q2 8 MHz, T1 MMBT2222A, U1 MPL3115A2, U2 MPU-9250, U3 ATMEGA328P_TQFP, U4 ADS1015

Commit message: mpu9250 stuff
Connections:
- net GND: now also U2.RESV2
- net LOGIC_VDD: now also U2.RESV
Changed lines of the file:
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@@
 <?xml version="1.0" encoding="utf-8"?>
 <!DOCTYPE eagle SYSTEM "eagle.dtd">
-<eagle version="7.5.0">
+<eagle version="7.6.0">
 <drawing>
 <settings>
@@
 <part name="MPWR1" library="SparkFun-Connectors" deviceset="M02" device="PTH" value="11.1"/>
 <part name="MPWR2" library="SparkFun-Connectors" deviceset="M02" device="PTH" value="7.4V"/>
+<part name="GND6" library="supply1" deviceset="GND" device=""/>
 </parts>
 <sheets>
@@
 <instance part="MPWR1" gate="G$1" x="203.2" y="243.84"/>
 <instance part="MPWR2" gate="G$1" x="203.2" y="208.28"/>
+<instance part="GND6" gate="1" x="-45.72" y="20.32"/>
 </instances>
 <busses>
@@
 <pinref part="C14" gate="G$1" pin="-"/>
 <pinref part="MPWR2" gate="G$1" pin="1"/>
+</segment>
+<segment>
+<pinref part="U2" gate="G$1" pin="RESV2"/>
+<wire x1="-53.34" y1="22.86" x2="-45.72" y2="22.86" width="0.1524" layer="91"/>
+<pinref part="GND6" gate="1" pin="GND"/>
 </segment>
 </net>
@@
 <label x="-101.6" y="15.24" size="1.778" layer="95" rot="R180" xref="yes"/>
 </segment>
-</net>
+<segment>
+<pinref part="U2" gate="G$1" pin="RESV"/>
+<wire x1="-99.06" y1="33.02" x2="-101.6" y2="33.02" width="0.1524" layer="91"/>
+<label x="-101.6" y="33.02" size="1.778" layer="95" rot="R180" xref="yes"/>
+</segment>
+</net>
