File: RCS/RCSfullschematic1.brd (EAGLE design)
At the start: 48.6 x 80 mm, 67 parts, among them IC1 ILD213T, IC2 FT232RL, J7 USB-MICROB, Q2 8 MHz, T1 MMBT2222A, U1 MPL3115A2, U2 MPU-9250, U3 ATMEGA328P_TQFP, U4 ADS1015

Commit message: changes to schematic
board is not ready yet
Parts:
- removed D3: 3A/600V, SparkFun-DiscreteSemi:SMA-DIODE_ALT
- removed IC1: ILD213T, SparkFun-DiscreteSemi:SO08
- added OK1: 4N35, optocoupler:DIL06
- F1, F2, F3, F4: device fuse:PICOFUSE -> SparkFun-PowerIC:PTC-1206
Connections:
- removed net N$4: D3.A, F1.1
- net 6V_POWER: now also F1.1; no longer D3.C
- net GND: now also OK1.2, U2.20; no longer IC1.2
- net GND1: now also OK1.4; no longer IC1.7
- net LOGIC_VDD: now also R6.2, R7.2, U2.19
- net N$2: now also OK1.5; no longer IC1.8
- net N$7: now also OK1.1; no longer IC1.1
- net VDD: no longer R6.2, R7.2
Routing:
- net N$4: track 6.41 -> 0.00 mm
- net N$17: track 53.4 -> 57.9 mm
- net N$21: track 58.0 -> 61.6 mm
- net VOUT-MOTOR: track 64.3 -> 67.9 mm
- net N$20: track 6.50 -> 10.1 mm
- net 6V_POWER: track 72.6 -> 74.8 mm
- net N$18: track 9.99 -> 7.98 mm
- net VCC: track 98.6 -> 96.8 mm
- net GND1: track 147.1 -> 145.9 mm

Commit message: mpu changes
Connections:
- removed net FSYNC: U2.11
- net GND: now also U2.11
- net LOGIC_VDD: now also U2.1
Changed lines of the file:
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@@
 <contactref element="U2" pad="20"/>
 <contactref element="OK1" pad="2"/>
+<contactref element="U2" pad="11"/>
 <wire x1="22.1742" y1="30.861" x2="21.92" y2="31.785" width="0" layer="19" extent="1-1"/>
+<wire x1="18.72" y1="31.785" x2="18.72" y2="32.585" width="0" layer="19" extent="1-1"/>
 <wire x1="-5.08" y1="3.175" x2="2.5146" y2="6.1722" width="0" layer="19" extent="1-1"/>
 </signal>
@@
 <wire x1="18.669" y1="31.3182" x2="18.72" y2="31.385" width="0.1524" layer="1"/>
 <wire x1="26.3652" y1="16.383" x2="26.41" y2="16.3576" width="0.1524" layer="1"/>
-</signal>
-<signal name="FSYNC">
-<contactref element="U2" pad="11"/>
 </signal>
 <signal name="N$1">
@@
 <contactref element="R6" pad="2"/>
 <contactref element="R7" pad="2"/>
+<contactref element="U2" pad="1"/>
 <wire x1="36.195" y1="33.172" x2="40.64" y2="33.172" width="0" layer="19" extent="1-1"/>
 <wire x1="30.5562" y1="31.7754" x2="36.195" y2="33.172" width="0" layer="19" extent="1-16"/>
+<wire x1="35.055" y1="26.67" x2="35.055" y2="26.67" width="0" layer="19" extent="1-16"/>
+<wire x1="21.32" y1="33.985" x2="19.2786" y2="32.766" width="0" layer="19" extent="1-1"/>
 <wire x1="21.92" y1="31.385" x2="20.574" y2="29.1846" width="0" layer="19" extent="1-1"/>
 </signal>

Commit message: changes?
Parts:
- added ERROR: Red, adafruit:CHIPLED_1206
- added R16: 100, adafruit:R1206
- D4: value 3A/600V -> BAT20JFILM; device SparkFun-DiscreteSemi:SMA-DIODE_ALT -> SparkFun-DiscreteSemi:SOD-323
- moved OK1 71.6 mm to (31.4, 68.6)
- moved D4 22.6 mm to (31.4, 60.3), turned to 0 degrees
- moved R2 19.7 mm to (16.5, 70.8)
- moved R3 19.2 mm to (40.0, 38.7), turned to 90 degrees
- moved C13 17.4 mm to (39.1, 46.4), turned to 270 degrees
- moved F1 15.8 mm to (31.8, 55.2), turned to 180 degrees
- moved C4 11.5 mm to (40.0, 32.4), turned to 270 degrees
- moved R1 10.2 mm to (38.7, 23.8)
- moved SERVO 10.2 mm to (38.1, 61.3)
- moved F3 10.1 mm to (16.5, 66.4)
- moved T1 9.42 mm to (38.7, 65.7)
- moved J6 9.21 mm to (7.30, 2.22)
- moved J1 8.58 mm to (28.9, 2.22)
- moved J7 8.25 mm to (2.54, 18.4)
- moved C12 7.94 mm to (23.5, 66.4)
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Connections:
- new net N$14: ERROR.C, R16.2
- new net N$23: ERROR.A, U3.2
- net GND: now also R16.1
Routing:
- net GND: track 406.2 -> 0.00 mm
- net GND1: track 145.9 -> 0.00 mm, vias 2 -> 0
- net LOGIC_VDD: track 144.4 -> 0.00 mm, vias 2 -> 0
- net A4(SDA): track 138.1 -> 0.00 mm, vias 3 -> 0
- net A5(SCL): track 127.2 -> 0.00 mm, vias 4 -> 0
- net VCC: track 96.8 -> 0.00 mm, vias 4 -> 0
- net FEEDBACK: track 81.3 -> 0.00 mm, vias 1 -> 0
- net MOTOR: track 75.6 -> 0.00 mm
- net 6V_POWER: track 74.8 -> 0.00 mm, vias 2 -> 0
- net VOUT-MOTOR: track 67.9 -> 0.00 mm
- net RESET: track 63.6 -> 0.00 mm, vias 3 -> 0
- net N$21: track 61.6 -> 0.00 mm
- net N$17: track 57.9 -> 0.00 mm, vias 1 -> 0
- net VDD: track 48.2 -> 0.00 mm
- net TX: track 41.8 -> 0.00 mm, vias 3 -> 0
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Other:
- board size 48.6 x 80 mm -> 43.2 x 80 mm
