File: RCS/RCSfullschematic1.sch (EAGLE design)
At the start: 67 parts, among them IC1 ILD213T, IC2 FT232RL, IC4 317T, J7 USB-MICROB, Q2 8 MHz, T1 MMBT2222A, U1 MPL3115A2, U2 MPU-9250, U3 ATMEGA328P_TQFP, U4 ADS1015

Commit message: SMASHED
Parts:
- removed IC4: 317T, linear:317T
- added IC3: (no value), v-reg:LM317TS
- F1, F4: value TRIP 1.5A -> 1.5A
- F3: value TRIP 100mA -> 100mA
Connections:
- net N$6 renamed SIGNAL
- net N$21: now also IC3.IN; no longer IC4.VI
- net N$22: now also IC3.ADJ; no longer IC4.ADJ
- net VOUT-MOTOR: now also IC3.OUT; no longer IC4.VO
Changed lines of the file:
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@@
 <part name="GND21" library="supply1" deviceset="GND" device=""/>
 <part name="D1" library="SparkFun-DiscreteSemi" deviceset="DIODE-ZENER" device="-BZT52C3V6S" value="3.3V"/>
-<part name="F3" library="fuse" deviceset="PICOFUSE" device="" value="TRIP 100mA"/>
+<part name="F3" library="fuse" deviceset="PICOFUSE" device="" value="100mA"/>
 <part name="GND" library="SparkFun-Aesthetics" deviceset="GND" device="" value=""/>
 <part name="JP1" library="SparkFun-Connectors" deviceset="M02" device="PTH" value="SENSOR/MCU"/>
@@
 <part name="LM117" library="SparkFun-IC-Power" deviceset="V_REG_LM1117" device="SOT223"/>
 <part name="SW3" library="special" deviceset="SW_DIP-1" device=""/>
-<part name="F4" library="fuse" deviceset="PICOFUSE" device="" value="TRIP 1.5A"/>
+<part name="F4" library="fuse" deviceset="PICOFUSE" device="" value="1.5A"/>
 <part name="C15" library="rcl" deviceset="C-US" device="C1206" value="0.1uF"/>
 <part name="C16" library="SparkFun-Capacitors" deviceset="10UF-POLAR" device="-EIA3216-16V-10%(TANT)" value="10uF"/>
@@
 <part name="R15" library="rcl" deviceset="R-US_" device="M1206" value="750"/>
 <part name="JP5" library="SparkFun-Connectors" deviceset="M02" device="PTH" value="MOTOR"/>
-<part name="F1" library="fuse" deviceset="PICOFUSE" device="" value="TRIP 1.5A"/>
+<part name="F1" library="fuse" deviceset="PICOFUSE" device="" value="1.5A"/>
 <part name="SUPPLY1" library="supply2" deviceset="GND1" device=""/>
 <part name="MPWR1" library="SparkFun-Connectors" deviceset="M02" device="PTH" value="11.1"/>
 <part name="MPWR2" library="SparkFun-Connectors" deviceset="M02" device="PTH" value="7.4V"/>
-<part name="IC4" library="linear" deviceset="*317" device="T"/>
+<part name="IC3" library="v-reg" deviceset="LM317TS" device=""/>
 </parts>
 <sheets>
@@
 <instance part="MPWR1" gate="G$1" x="203.2" y="243.84"/>
 <instance part="MPWR2" gate="G$1" x="203.2" y="208.28"/>
-<instance part="IC4" gate="A1" x="312.42" y="254"/>
+<instance part="IC3" gate="1" x="312.42" y="256.54"/>
 </instances>
 <busses>
@@
 </segment>
 </net>
-<net name="N$6" class="1">
+<net name="SIGNAL" class="1">
 <segment>
 <pinref part="T1" gate="G$1" pin="C"/>
@@
 <pinref part="C16" gate="G$1" pin="+"/>
 <wire x1="292.1" y1="256.54" x2="292.1" y2="248.92" width="0.1524" layer="91"/>
-<pinref part="IC4" gate="A1" pin="VI"/>
-<wire x1="292.1" y1="256.54" x2="302.26" y2="256.54" width="0.1524" layer="91"/>
+<wire x1="292.1" y1="256.54" x2="304.8" y2="256.54" width="0.1524" layer="91"/>
 <junction x="292.1" y="256.54"/>
+<pinref part="IC3" gate="1" pin="IN"/>
 </segment>
 </net>
@@
 <wire x1="312.42" y1="241.3" x2="312.42" y2="238.76" width="0.1524" layer="91"/>
 <wire x1="327.66" y1="241.3" x2="312.42" y2="241.3" width="0.1524" layer="91"/>
-<pinref part="IC4" gate="A1" pin="ADJ"/>
 <wire x1="312.42" y1="248.92" x2="312.42" y2="241.3" width="0.1524" layer="91"/>
 <junction x="312.42" y="241.3"/>
+<pinref part="IC3" gate="1" pin="ADJ"/>
 </segment>
 </net>
@@
 <junction x="337.82" y="256.54"/>
 <label x="355.6" y="256.54" size="1.27" layer="95" xref="yes"/>
-<pinref part="IC4" gate="A1" pin="VO"/>
-<wire x1="322.58" y1="256.54" x2="327.66" y2="256.54" width="0.1524" layer="91"/>
+<wire x1="320.04" y1="256.54" x2="327.66" y2="256.54" width="0.1524" layer="91"/>
 <junction x="327.66" y="256.54"/>
-</segment>
-<segment>
+<pinref part="IC3" gate="1" pin="OUT"/>
+</segment>
+<segment>

Commit message: cool beans
Connections:
- new net N$6: R11.1, U4.ADDR
- net A4(SDA): no longer R11.1, U4.ADDR
Changed lines of the file:
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@@
-</segment>
-<segment>
-<pinref part="U4" gate="G$1" pin="ADDR"/>
-<pinref part="R11" gate="G$1" pin="1"/>
-<wire x1="518.16" y1="132.08" x2="530.86" y2="132.08" width="0.1524" layer="91"/>
 </segment>
 <segment>
@@
 </segment>
 </net>
+<net name="N$6" class="0">
+<segment>
+<pinref part="U4" gate="G$1" pin="ADDR"/>
+<pinref part="R11" gate="G$1" pin="1"/>
+<wire x1="518.16" y1="132.08" x2="530.86" y2="132.08" width="0.1524" layer="91"/>
+</segment>
+</net>
 </nets>
 </sheet>
 </sheets>
+<errors>
+</errors>
 </schematic>
 </drawing>

Commit message: changes to schematic
board is not ready yet
Parts:
- removed D3: 3A/600V, SparkFun-DiscreteSemi:DIODESMA-ALT
- removed IC1: ILD213T, SparkFun-DiscreteSemi:ILD213T
- added OK1: 4N35, optocoupler:4N35
- F1, F2, F3, F4: device fuse:PICOFUSE -> SparkFun-PowerIC:PTCSMD
Connections:
- removed net N$4: D3.A, F1.1
- net 6V_POWER: now also F1.1; no longer D3.C
- net GND: now also OK1.C, U2.RESV2; no longer IC1.C1
- net GND1: now also OK1.EMI; no longer IC1.ET2
- net LOGIC_VDD: now also R6.2, R7.2, U2.RESV1
- net N$2: now also OK1.COL; no longer IC1.CT2
- net N$7: now also OK1.A; no longer IC1.A1
- net VDD: no longer R6.2, R7.2
Other:
- moved on the sheet: R1

Commit message: mpu changes
Connections:
- removed net FSYNC: U2.FSYNC
- net GND: now also U2.FSYNC
- net LOGIC_VDD: now also U2.RESV
Changed lines of the file:
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@@
 <pinref part="MPWR2" gate="G$1" pin="1"/>
+</segment>
+<segment>
+<pinref part="U2" gate="G$1" pin="FSYNC"/>
+<wire x1="-99.06" y1="7.62" x2="-101.6" y2="7.62" width="0.1524" layer="91"/>
+<label x="-101.6" y="7.62" size="1.778" layer="95" rot="R180" xref="yes"/>
 </segment>
 </net>
@@
 <wire x1="502.92" y1="45.72" x2="505.46" y2="45.72" width="0.1524" layer="91"/>
 <label x="505.46" y="45.72" size="1.27" layer="95" xref="yes"/>
-</segment>
-</net>
-<net name="FSYNC" class="0">
-<segment>
-<pinref part="U2" gate="G$1" pin="FSYNC"/>
-<wire x1="-99.06" y1="7.62" x2="-101.6" y2="7.62" width="0.1524" layer="91"/>
-<label x="-101.6" y="7.62" size="1.778" layer="95" rot="R180" xref="yes"/>
 </segment>
 </net>
@@
 <label x="581.66" y="83.82" size="1.778" layer="95" xref="yes"/>
 </segment>
-</net>
+<segment>
+<pinref part="U2" gate="G$1" pin="RESV"/>
+<wire x1="-99.06" y1="33.02" x2="-106.68" y2="33.02" width="0.1524" layer="91"/>
+<label x="-106.68" y="33.02" size="1.778" layer="95" rot="R180" xref="yes"/>
+</segment>
+</net>

Commit message: changes?
Parts:
- added ERROR: Red, adafruit:LEDCHIPLED_1206
- added R16: 100, adafruit:R-US_R1206
- D4: value 3A/600V -> BAT20JFILM; device SparkFun-DiscreteSemi:DIODESMA-ALT -> SparkFun-DiscreteSemi:BAT20JFILM
Connections:
- new net N$14: ERROR.C, R16.2
- new net N$23: ERROR.A, U3.PD4(XCK/T0)
- net GND: now also R16.1
Changed lines of the file:
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@@
 <part name="C4" library="SparkFun-Passives" deviceset="CAP" device="1206" value="0.1uF"/>
 <part name="C5" library="SparkFun-Passives" deviceset="CAP" device="1206" value="0.1uF"/>
-<part name="D4" library="SparkFun-DiscreteSemi" deviceset="DIODE" device="SMA-ALT" value="3A/600V"/>
+<part name="D4" library="SparkFun-DiscreteSemi" deviceset="BAT20JFILM" device="" value="BAT20JFILM"/>
 <part name="R1" library="SparkFun-Passives" deviceset="RESISTOR" device="1206" value="220"/>
 <part name="R2" library="SparkFun-Passives" deviceset="RESISTOR" device="1206" value="10k"/>
@@
 <part name="IC3" library="v-reg" deviceset="LM317TS" device=""/>
 <part name="OK1" library="optocoupler" deviceset="4N35" device=""/>
+<part name="ERROR" library="adafruit" deviceset="LED" device="CHIPLED_1206" value="Red"/>
+<part name="R16" library="adafruit" deviceset="R-US_" device="R1206" value="100"/>
 </parts>
 <sheets>
@@
 <instance part="IC3" gate="1" x="312.42" y="256.54"/>
 <instance part="OK1" gate="G$1" x="160.02" y="76.2" rot="R270"/>
+<instance part="ERROR" gate="G$1" x="508" y="33.02" smashed="yes">
+<attribute name="NAME" x="511.556" y="28.448" size="1.778" layer="95" rot="R90"/>
+<attribute name="VALUE" x="513.715" y="28.448" size="1.778" layer="96" rot="R90"/>
+</instance>
+<instance part="R16" gate="G$1" x="502.92" y="5.08" rot="R90"/>
 </instances>
 <busses>
@@
 <pinref part="R10" gate="G$1" pin="1"/>
 <pinref part="GND16" gate="1" pin="GND"/>
-<wire x1="510.54" y1="0" x2="510.54" y2="-5.08" width="0.1524" layer="91"/>
+<wire x1="510.54" y1="0" x2="510.54" y2="-2.54" width="0.1524" layer="91"/>
+<pinref part="R16" gate="G$1" pin="1"/>
+<wire x1="510.54" y1="-2.54" x2="510.54" y2="-5.08" width="0.1524" layer="91"/>
+<wire x1="502.92" y1="0" x2="502.92" y2="-2.54" width="0.1524" layer="91"/>
+<wire x1="502.92" y1="-2.54" x2="510.54" y2="-2.54" width="0.1524" layer="91"/>
+<junction x="510.54" y="-2.54"/>
 </segment>
 <segment>
@@
 </segment>
 </net>
+<net name="N$14" class="0">
+<segment>
+<pinref part="R16" gate="G$1" pin="2"/>
+<wire x1="502.92" y1="10.16" x2="508" y2="10.16" width="0.1524" layer="91"/>
+<pinref part="ERROR" gate="G$1" pin="C"/>
+<wire x1="508" y1="10.16" x2="508" y2="27.94" width="0.1524" layer="91"/>
+</segment>
+</net>
+<net name="N$23" class="0">
+<segment>
+<pinref part="ERROR" gate="G$1" pin="A"/>
+<wire x1="508" y1="35.56" x2="508" y2="40.64" width="0.1524" layer="91"/>
+<pinref part="U3" gate="U$1" pin="PD4(XCK/T0)"/>
+<wire x1="508" y1="40.64" x2="502.92" y2="40.64" width="0.1524" layer="91"/>
+</segment>
+</net>
